Commit message: Add files via upload

File: SLDASM/urdf/SLDASM.urdf (robot description, URDF)
Before this commit: robot SLDASM, 4 links, 3 joints
Links:
- link link_2: mass 0.735688332874957 -> 0.735688332874956
- link link_3: mass 0.454304812581279 -> 0.460587997888459
Joints:
- joint joint_1: limit lower=0 upper=0 effort=0 velocity=0 -> lower=0 upper=0.03 effort=0 velocity=0; origin xyz=0.0066366 -0.42337 -0.025756 rpy=1.5708 0 0 -> xyz=0.0066366 -0.563 -0.025756 rpy=1.5708 0 0; type revolute -> prismatic
- joint joint_2: origin xyz=0 -0.20072 0.012 rpy=0 0 -1.1868 -> xyz=0 -0.200720396700335 0.012 rpy=0 0 0.995527576712073
- joint joint_3: origin xyz=0 -0.25 0 rpy=0 0 1.9202 -> xyz=0 -0.25 0 rpy=0 0 -0.995527576712073
